File: TypeC2DoubleVoltage.kicad_pcb (KiCad board)
At the start: 2 copper layers, 66 x 35.6 mm, 66 parts, among them J1 USB_C_Receptacle_PowerOnly_6P, J2 SMA-KE, J3 SMA-KE, U1 MC34063AD, U2 LM317_SOT-223, U3 MC34063AD, U4 LM337_SOT223

Commit message: Update
Parts:
- removed C23, C30: 104 0402 50V X7R, Capacitor_SMD:C_0402_1005Metric
- removed C24, C29: 105 0402 25V X5R, Capacitor_SMD:C_0402_1005Metric
- removed C25: NPXC0421E470MF, Capacitor_THT:CP_Radial_D6.3mm_P2.50mm
- removed C26: 10uF 25V D4xL5, Capacitor_THT:CP_Radial_D4.0mm_P1.50mm
- removed C27, C28: 100uF 16V D6.3xL5, Capacitor_THT:CP_Radial_D6.3mm_P2.50mm
- removed J2, J3: SMA-KE, Customer_Connector:SMA-KE_1.6mm
- added D4: K24-MS, Diode_SMD:D_SOD-123F, F.Cu at (168.0, 81.7)
- C1, C14, C16: value 105 0402 25V X5R -> 105 0603 25V X5R; footprint Capacitor_SMD:C_0402_1005Metric -> Capacitor_SMD:C_0603_1608Metric
- C10: value NPXC0421E470MF -> 10uF 16V D4xL5; footprint Capacitor_THT:CP_Radial_D6.3mm_P2.50mm -> Capacitor_THT:CP_Radial_D4.0mm_P1.50mm
- C11: value 10uF 25V D4xL5 -> 220uF 16V D8xL5; footprint Capacitor_THT:CP_Radial_D4.0mm_P1.50mm -> Capacitor_THT:CP_Radial_D8.0mm_P3.50mm
- C12: value 100uF 16V D6.3xL5 -> 105 0603 25V X5R; footprint Capacitor_THT:CP_Radial_D6.3mm_P2.50mm -> Capacitor_SMD:C_0603_1608Metric
- C13: value 100uF 16V D6.3xL5 -> 100uF 10V D5xL5; footprint Capacitor_THT:CP_Radial_D6.3mm_P2.50mm -> Capacitor_THT:CP_Radial_D4.0mm_P2.00mm
- C15: value 104 0402 50V X7R -> 331 0603 50V X7R; footprint Capacitor_SMD:C_0402_1005Metric -> Capacitor_SMD:C_0603_1608Metric
- C17, C6: value 105 0402 25V X5R -> 100uF 16V D6.3xL5; footprint Capacitor_SMD:C_0402_1005Metric -> Capacitor_THT:CP_Radial_D6.3mm_P2.50mm
- C18: value 220uF 10V D6.3xL5 -> 100uF 16V D6.3xL5
- C19: value 181 0402 50V X7R -> 220uF 16V D8xL5; footprint Capacitor_SMD:C_0402_1005Metric -> Capacitor_THT:CP_Radial_D8.0mm_P3.50mm
- C2: value 105 0402 25V X5R -> 100uF 10V D5xL5; footprint Capacitor_SMD:C_0402_1005Metric -> Capacitor_THT:CP_Radial_D4.0mm_P2.00mm
- C20: value NPXC0421E470MF -> 220uF 16V D8xL5; footprint Capacitor_THT:CP_Radial_D6.3mm_P2.50mm -> Capacitor_THT:CP_Radial_D8.0mm_P3.50mm
- C21: value 105 0402 25V X5R -> 10uF 16V D4xL5; footprint Capacitor_SMD:C_0402_1005Metric -> Capacitor_THT:CP_Radial_D4.0mm_P1.50mm
- C22, C8: value 104 0402 50V X7R -> 220uF 16V D8xL5; footprint Capacitor_SMD:C_0402_1005Metric -> Capacitor_THT:CP_Radial_D8.0mm_P3.50mm
- C3: value 220uF 10V D6.3xL5 -> 105 0603 25V X5R; footprint Capacitor_THT:CP_Radial_D6.3mm_P2.50mm -> Capacitor_SMD:C_0603_1608Metric
- C4: value 181 0402 50V X7R -> 331 0603 50V X7R; footprint Capacitor_SMD:C_0402_1005Metric -> Capacitor_SMD:C_0603_1608Metric
- C5: value NPXC0421E470MF -> 105 0603 25V X5R; footprint Capacitor_THT:CP_Radial_D6.3mm_P2.50mm -> Capacitor_SMD:C_0603_1608Metric
- C7: value 104 0402 50V X7R -> 100uF 16V D6.3xL5; footprint Capacitor_SMD:C_0402_1005Metric -> Capacitor_THT:CP_Radial_D6.3mm_P2.50mm
- C9: value 105 0402 25V X5R -> 220uF 16V D8xL5; footprint Capacitor_SMD:C_0402_1005Metric -> Capacitor_THT:CP_Radial_D8.0mm_P3.50mm
- D1: value LED 0402 -> LED 0603; footprint LED_SMD:LED_0402_1005Metric -> LED_SMD:LED_0603_1608Metric
- D2: value K24-MS -> PESD5V0 SOD-523; footprint Diode_SMD:D_SOD-123F -> Diode_SMD:D_SOD-523
- J1: footprint Connector_USB:USB_C_Receptacle_GCT_USB4135-GF-A_6P_TopMnt_Horizontal -> Customer_Connector:USB_C_Receptacle_6P_01
- L1, L5: value 18uH 3015 -> 22uH 3015
- L2, L6: value 22uH 5040 -> 47uH 4030; footprint Inductor_SMD:L_Changjiang_FNR5040S -> Inductor_SMD:L_Changjiang_FNR4030S
- L3, L7: value 150uH 3015 -> 100uH 3015
- L4, L8: value 18uH 3015 -> 100uH 3015
- R1, R2: value 5.1k 0402 -> 5.1k 0603; footprint Resistor_SMD:R_0402_1005Metric -> Resistor_SMD:R_0603_1608Metric
- R10, R4: value 200mR 1210 -> 300mR 1206; footprint Resistor_SMD:R_1210_3225Metric -> Resistor_SMD:R_1206_3216Metric
- R11, R14, R3, R7, R8: value 1k 0402 -> 1k 0603; footprint Resistor_SMD:R_0402_1005Metric -> Resistor_SMD:R_0603_1608Metric
- R12, R6: value 11k 0402 -> 10.2k 0603; footprint Resistor_SMD:R_0402_1005Metric -> Resistor_SMD:R_0603_1608Metric
- R13, R9: value 8.25k 0402 -> 8.25k 0603; footprint Resistor_SMD:R_0402_1005Metric -> Resistor_SMD:R_0603_1608Metric
- R5: value 180R 1206 -> 180R 0603; footprint Resistor_SMD:R_1206_3216Metric -> Resistor_SMD:R_0603_1608Metric
- moved H2 99.6 mm to (147.6, 45.5)
- moved C8 92.8 mm to (137.1, 38.3), turned to 0 degrees
- moved L1 92.6 mm to (161.9, 35.9), turned to 0 degrees
- moved H1 88.1 mm to (147.6, 37.5)
- moved C9 86.1 mm to (137.1, 47.9), turned to 0 degrees
- moved C1 83.3 mm to (145.6, 66.6), turned to 0 degrees
- moved C6 78.4 mm to (154.4, 37.5)
- moved C3 76.8 mm to (145.6, 69.1), turned to 0 degrees
- moved L3 76.3 mm to (161.9, 40.5), turned to 0 degrees
- moved J1 74.3 mm to (149.2, 80.0), turned to 0 degrees
- moved C7 72.5 mm to (154.4, 45.3)
- moved U2 70.9 mm to (169.1, 37.7), turned to 0 degrees
- moved R1 69.9 mm to (149.7, 74.1), turned to 0 degrees
- moved C17 69.8 mm to (154.4, 53.2), turned to 0 degrees
- moved C11 69.4 mm to (137.1, 57.4), turned to 0 degrees
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Connections:
- C10 pad 1: Net-(C10-Pad1) -> Net-(U2-ADJ)
- C11 pad 1: Net-(U2-ADJ) -> +12V
- C12 pad 1: +12V -> GNDREF
- C12 pad 2: GNDREF -> VCC
- C13 pad 1: +12V -> /U3_Vin
- C14 pad 2: +12V -> /U3_Vin
- C15 pad 1: GNDREF -> /U3_Vout
- C15 pad 2: +12V -> Net-(U3-TC)
- C16 pad 1: GNDREF -> /U3_Vout
- C16 pad 2: VCC -> GNDREF
- C17 pad 2: /U3_Vin -> /U3_Vout
- C18 pad 1: /U3_Vin -> GNDREF
- C18 pad 2: GNDREF -> Net-(C18-Pad2)
- C19 pad 1: /U3_Vout -> GNDREF
- C19 pad 2: Net-(U3-TC) -> /U4_Vin
- C2 pad 1: GNDREF -> /U1_Vin
- C2 pad 2: /U1_Vin -> GNDREF
- C20 pad 2: /U3_Vout -> /U4_Vin
- C21 pad 1: /U3_Vout -> GNDREF
- C21 pad 2: GNDREF -> Net-(U4-ADJ)
- C22 pad 1: /U3_Vout -> GNDREF
- C22 pad 2: GNDREF -> -12V
- C3 pad 1: /U1_Vin -> GNDREF
- C3 pad 2: GNDREF -> /U1_Vin
- C5 pad 1: /U1_Vout -> GNDREF
- C5 pad 2: GNDREF -> /U1_Vout
- C6 pad 1: GNDREF -> /U1_Vout
- C6 pad 2: /U1_Vout -> GNDREF
- C7 pad 1: GNDREF -> Net-(C7-Pad1)
- C7 pad 2: /U1_Vout -> GNDREF
- C8 pad 1: GNDREF -> /U2_Vin
- C8 pad 2: Net-(C10-Pad1) -> GNDREF
- C9 pad 1: GNDREF -> /U2_Vin
- C9 pad 2: Net-(C10-Pad1) -> GNDREF
- D2 pad 1: /U1_Vout -> GNDREF
- D2 pad 2: Net-(D2-A) -> VCC
- D3 pad 1: Net-(D3-K) -> /U1_Vout
- D3 pad 2: /U3_Vout -> Net-(D3-A)
- L2 pad 2: Net-(D2-A) -> Net-(D3-A)
- L3 pad 2: Net-(C10-Pad1) -> Net-(C7-Pad1)
- L4 pad 1: Net-(C10-Pad1) -> Net-(C7-Pad1)
- L6 pad 1: Net-(D3-K) -> Net-(D4-K)
- L7 pad 2: Net-(C23-Pad1) -> Net-(C18-Pad2)
- L8 pad 1: Net-(C23-Pad1) -> Net-(C18-Pad2)
- R12 pad 1: GNDREF -> Net-(U3-Vfb)
- R12 pad 2: /U3_Vout -> GNDREF
- U1 pad 1: Net-(D2-A) -> Net-(D3-A)
- U3 pad 2: Net-(D3-K) -> Net-(D4-K)
Routing:
- net Net-(U1-Vfb): track 12.9 -> 0.00 mm
- net Net-(U2-ADJ): track 10.9 -> 0.00 mm
- net Net-(U1-Ipk): track 10.0 -> 0.00 mm
- net /U3_Vout: track 9.65 -> 0.00 mm
- net Net-(U4-ADJ): track 8.33 -> 0.00 mm
- net Net-(U1-DC): track 3.81 -> 0.00 mm
- net Net-(J1-CC1): track 2.86 -> 0.00 mm
- net Net-(J1-CC2): track 2.86 -> 0.00 mm
- net Net-(U3-TC): track 2.03 -> 0.00 mm
- net Net-(U1-TC): track 1.97 -> 0.00 mm
- net Net-(U3-Vfb): track 1.93 -> 0.00 mm
- net /U1_Vout: track 1.91 -> 0.00 mm
- net Net-(D1-K): track 1.54 -> 0.00 mm
- net GNDREF: vias 94 -> 0
- removed copper zone on F.Cu, net +12V
- removed copper zone on F.Cu, net -12V
- removed copper zone on F.Cu, net /U1_Vin
- removed copper zone on F.Cu, net /U1_Vout
- removed copper zone on F.Cu, net /U2_Vin
- removed copper zone on F.Cu, net /U3_Vin
- removed copper zone on F.Cu, net /U3_Vout
- removed copper zone on F.Cu, net /U4_Vin
- removed copper zone on B.Cu, net GNDREF
- removed copper zone on F.Cu, net GNDREF
- removed copper zone on F.Cu, net Net-(C10-Pad1)
- removed copper zone on F.Cu, net Net-(C23-Pad1)
- removed copper zone on F.Cu, net Net-(D2-A)
- removed copper zone on F.Cu, net Net-(D3-K)
- removed copper zone on F.Cu, net Net-(U1-Ipk)
- removed copper zone on F.Cu, net Net-(U3-DC)
- removed copper zone on F.Cu, net VCC
Other:
- board outline removed
- board text removed: "V+"
- board text removed: "V-"

Commit message: Almost Finish
Parts:
- removed D2: PESD5V0 SOD-523, Diode_SMD:D_SOD-523
- added J2: Conn_01x10_Pin, Connector_PinHeader_2.54mm:PinHeader_1x10_P2.54mm_Horizontal, F.Cu at (176.8, 123.4)
- C11, C19, C20, C22, C8, C9: value 220uF 16V D8xL5 -> 100uF 16V D6.3xL5; footprint Capacitor_THT:CP_Radial_D8.0mm_P3.50mm -> Capacitor_THT:CP_Radial_D6.3mm_P2.50mm
- moved H2 119.4 mm to (239.1, 122.2)
- moved H1 111.8 mm to (239.1, 101.9)
- moved L1 99.8 mm to (233.2, 105.7), turned to 180 degrees
- moved C12 99.4 mm to (235.8, 118.4), turned to 180 degrees
- moved C1 98.3 mm to (234.0, 109.6), turned to 90 degrees
- moved R3 97.6 mm to (233.9, 122.2), turned to -90 degrees
- moved C14 96.8 mm to (228.9, 122.2), turned to 90 degrees
- moved L5 96.7 mm to (230.1, 118.4), turned to 180 degrees
- moved C3 95.4 mm to (232.0, 109.6), turned to 90 degrees
- moved C8 95.1 mm to (207.9, 101.9), turned to 90 degrees
- moved J1 94.2 mm to (237.8, 112.0), turned to 90 degrees
- moved C9 93.9 mm to (207.9, 109.5), turned to 180 degrees
- moved R1 91.7 mm to (232.4, 113.6), turned to 180 degrees
- moved R2 91.3 mm to (232.4, 115.2), turned to 180 degrees
- moved C17 90.1 mm to (209.2, 124.7), turned to 90 degrees
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Connections:
- D1 pad 1: Net-(D1-K) -> GNDREF
- D1 pad 2: VCC -> Net-(D1-A)
- R3 pad 1: Net-(D1-K) -> VCC
- R3 pad 2: GNDREF -> Net-(D1-A)
Routing:
- net Net-(U1-Vfb): track 0.00 -> 17.3 mm
- net Net-(U2-ADJ): track 0.00 -> 14.0 mm
- net -12V: track 0.00 -> 10.2 mm
- net Net-(U4-ADJ): track 0.00 -> 9.44 mm
- net Net-(J1-CC1): track 0.00 -> 6.05 mm
- net +12V: track 0.00 -> 5.72 mm
- net Net-(J1-CC2): track 0.00 -> 5.44 mm
- net Net-(U3-Vfb): track 0.00 -> 5.21 mm
- net Net-(U1-Ipk): track 0.00 -> 4.68 mm
- net Net-(U3-TC): track 0.00 -> 2.54 mm
- net Net-(U1-TC): track 0.00 -> 2.54 mm
- net /U1_Vout: track 0.00 -> 2.48 mm
- net Net-(U1-DC): track 0.00 -> 1.91 mm
- net /U3_Vout: track 0.00 -> 1.91 mm
- net Net-(D1-A): track 0.00 -> 1.75 mm
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- added copper zone on F.Cu, net +12V
- added copper zone on F.Cu, net -12V
- added copper zone on F.Cu, net /U1_Vin
- added copper zone on F.Cu, net /U1_Vout
- added copper zone on F.Cu, net /U2_Vin
- added copper zone on F.Cu, net /U3_Vin
- added copper zone on F.Cu, net /U3_Vout
- added copper zone on F.Cu, net /U4_Vin
- added copper zone on B.Cu, net GNDREF
- added copper zone on F.Cu, net GNDREF
- added copper zone on F.Cu, net Net-(C18-Pad2)
- added copper zone on F.Cu, net Net-(C7-Pad1)
- added copper zone on F.Cu, net Net-(D3-A)
- added copper zone on F.Cu, net Net-(D4-K)
- added copper zone on F.Cu, net Net-(U1-Ipk)
- added copper zone on F.Cu, net Net-(U3-DC)
- added copper zone on F.Cu, net VCC
Other:
- board outline added: 71.1 x 30.5 mm
- board text added: "+Vout"
- board text added: "-Vout"
- board text added: "GND"

Commit message: Update
Parts:
- removed C18, C20: 100uF 16V D6.3xL5, Capacitor_THT:CP_Radial_D6.3mm_P2.50mm
- C11, C19, C22, C8: value 100uF 16V D6.3xL5 -> 47uF 16V D5xL5; footprint Capacitor_THT:CP_Radial_D6.3mm_P2.50mm -> Capacitor_THT:CP_Radial_D5.0mm_P2.00mm
- C13, C2: value 100uF 10V D5xL5 -> 106 0805 25V X5R; footprint Capacitor_THT:CP_Radial_D4.0mm_P2.00mm -> Capacitor_SMD:C_0805_2012Metric
- C14: value 105 0603 25V X5R -> 106 0805 25V X5R; footprint Capacitor_SMD:C_0603_1608Metric -> Capacitor_SMD:C_0805_2012Metric
- C17, C6, C7: value 100uF 16V D6.3xL5 -> 106 0805 25V X5R; footprint Capacitor_THT:CP_Radial_D6.3mm_P2.50mm -> Capacitor_SMD:C_0805_2012Metric
- C9: value 100uF 16V D6.3xL5 -> 105 0603 25V X5R; footprint Capacitor_THT:CP_Radial_D6.3mm_P2.50mm -> Capacitor_SMD:C_0603_1608Metric
- J2: footprint Connector_PinHeader_2.54mm:PinHeader_1x10_P2.54mm_Horizontal -> Connector_PinHeader_2.54mm:PinHeader_1x10_P2.54mm_Vertical
- R10, R4: value 300mR 1206 -> 200mR 1206
- R11, R7: value 1k 0603 -> 499R 0603
- R12, R6: value 10.2k 0603 -> 5.1k 0603
- R13, R9: value 8.25k 0603 -> 5.1k 0603
- R14, R8: value 1k 0603 -> 604R 0603
- moved H2 164.2 mm to (76.5, 99.3)
- moved H1 163.8 mm to (76.5, 81.5)
- moved C3 135.1 mm to (98.7, 87.7)
- moved C14 132.9 mm to (97.8, 100.6), turned to -90 degrees
- moved R7 121.5 mm to (112.8, 90.4)
- moved C7 121.4 mm to (99.4, 80.9), turned to 180 degrees
- moved D1 120.9 mm to (114.5, 92.1)
- moved R3 120.7 mm to (116.8, 93.0), turned to 90 degrees
- moved C1 120.6 mm to (117.0, 80.3), turned to -90 degrees
- moved C12 120.4 mm to (116.8, 99.9), turned to 90 degrees
- moved J1 119.8 mm to (120.0, 90.4)
- moved C2 119.5 mm to (114.6, 87.9)
- moved U1 119.4 mm to (109.5, 86.6)
- moved L1 119.3 mm to (115.9, 84.1)
- moved C4 119.2 mm to (104.8, 88.0)
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Connections:
- C13 pad 1: /U3_Vin -> GNDREF
- C13 pad 2: GNDREF -> /U3_Vin
- C14 pad 1: GNDREF -> /U3_Vout
- C14 pad 2: /U3_Vin -> GNDREF
- C17 pad 1: GNDREF -> Net-(C17-Pad1)
- C17 pad 2: /U3_Vout -> GNDREF
- C2 pad 1: /U1_Vin -> GNDREF
- C2 pad 2: GNDREF -> /U1_Vin
- C3 pad 2: /U1_Vin -> Net-(C3-Pad2)
- C6 pad 1: /U1_Vout -> GNDREF
- C6 pad 2: GNDREF -> /U1_Vout
- C7 pad 1: Net-(C7-Pad1) -> GNDREF
- C7 pad 2: GNDREF -> Net-(C3-Pad2)
- C9 pad 1: /U2_Vin -> Net-(C17-Pad1)
- L3 pad 2: Net-(C7-Pad1) -> Net-(C3-Pad2)
- L4 pad 1: Net-(C7-Pad1) -> Net-(C3-Pad2)
- L7 pad 2: Net-(C18-Pad2) -> Net-(C17-Pad1)
- L8 pad 1: Net-(C18-Pad2) -> Net-(C17-Pad1)
Routing:
- net +12V: track 5.72 -> 24.0 mm
- net -12V: track 10.2 -> 25.1 mm
- net Net-(U1-Vfb): track 17.3 -> 3.68 mm
- net GNDREF: track 0.00 -> 13.2 mm, vias 62 -> 120
- net Net-(U2-ADJ): track 14.0 -> 8.30 mm
- net /U1_Vout: track 2.48 -> 7.75 mm
- net Net-(U1-Ipk): track 4.68 -> 0.00 mm
- net Net-(J1-CC1): track 6.05 -> 3.19 mm
- net Net-(U3-Vfb): track 5.21 -> 7.72 mm
- net /U3_Vout: track 1.91 -> 0.00 mm
- net VCC: track 1.52 -> 0.00 mm
- net Net-(U4-ADJ): track 9.44 -> 7.95 mm
- net Net-(U1-DC): track 1.91 -> 2.82 mm
- added copper zone on B.Cu, net /U2_Vin
- added copper zone on F.Cu, net Net-(C17-Pad1)
- added copper zone on F.Cu, net Net-(C3-Pad2)
- removed copper zone on F.Cu, net -12V
- removed copper zone on F.Cu, net Net-(C18-Pad2)
- removed copper zone on F.Cu, net Net-(C7-Pad1)
Other:
- board size 71.1 x 30.5 mm -> 55.9 x 25.4 mm
- board text added: "V+"
- board text added: "V-"
- board text removed: "+Vout"
- board text removed: "-Vout"
