File: TypeC2DoubleVoltage.kicad_sch (KiCad schematic)
At the start: 59 parts, among them J1 USB_C_Receptacle_PowerOnly_6P, J2 15EDGR-3.5_2P, J3 15EDGR-3.5_2P, J4 15EDGR-3.5_2P, U1 MC34063AD, U2 LM317_SOT-223, U3 MC34063AD, U4 LM337_SOT223

Commit message: Update
Parts:
- removed C12: 100uF 16V D6.3xL5, Capacitor_THT:CP_Radial_D6.3mm_P2.50mm, symbol Device:C_Polarized
- removed J2, J3, J4: 15EDGR-3.5_2P, symbol Connector:Screw_Terminal_01x02
- added C11: 220uF 16V D8xL5, Capacitor_THT:CP_Radial_D8.0mm_P3.50mm, symbol Device:C_Polarized
- added D2: PESD5V0 SOD-523, Diode_SMD:D_SOD-523, symbol Device:D_TVS
- C1, C4: footprint Capacitor_SMD:C_0402_1005Metric -> Capacitor_SMD:C_0603_1608Metric
- C10: renamed from C11; value 10uF 16V D3xL5 -> 10uF 16V D4xL5
- C12: renamed from C16; footprint Capacitor_SMD:C_0402_1005Metric -> Capacitor_SMD:C_0603_1608Metric
- C13: renamed from C18; footprint Capacitor_THT:CP_Radial_D6.3mm_P2.50mm -> Capacitor_THT:CP_Radial_D4.0mm_P2.00mm
- C14: renamed from C9; footprint Capacitor_SMD:C_0402_1005Metric -> Capacitor_SMD:C_0603_1608Metric
- C15: renamed from C19; footprint Capacitor_SMD:C_0402_1005Metric -> Capacitor_SMD:C_0603_1608Metric
- C16: renamed from C21; footprint Capacitor_SMD:C_0402_1005Metric -> Capacitor_SMD:C_0603_1608Metric
- C19: renamed from C14; footprint Capacitor_THT:CP_Radial_D6.3mm_P2.50mm -> Capacitor_THT:CP_Radial_D8.0mm_P3.50mm
- C2: renamed from C3; footprint Capacitor_THT:CP_Radial_D6.3mm_P2.50mm -> Capacitor_THT:CP_Radial_D4.0mm_P2.00mm
- C20: renamed from C15; footprint Capacitor_THT:CP_Radial_D6.3mm_P2.50mm -> Capacitor_THT:CP_Radial_D8.0mm_P3.50mm
- C21: renamed from C10; value 10uF 16V D3xL5 -> 10uF 16V D4xL5
- C22: renamed from C17; footprint Capacitor_THT:CP_Radial_D6.3mm_P2.50mm -> Capacitor_THT:CP_Radial_D8.0mm_P3.50mm
- C3: renamed from C8; footprint Capacitor_SMD:C_0402_1005Metric -> Capacitor_SMD:C_0603_1608Metric
- C5: renamed from C6; footprint Capacitor_SMD:C_0402_1005Metric -> Capacitor_SMD:C_0603_1608Metric
- C8: renamed from C22; footprint Capacitor_THT:CP_Radial_D6.3mm_P2.50mm -> Capacitor_THT:CP_Radial_D8.0mm_P3.50mm
- C9: renamed from C23; footprint Capacitor_THT:CP_Radial_D6.3mm_P2.50mm -> Capacitor_THT:CP_Radial_D8.0mm_P3.50mm
- D1: footprint LED_SMD:LED_0402_1005Metric -> LED_SMD:LED_0603_1608Metric
- J1: footprint Connector_USB:USB_C_Receptacle_GCT_USB4135-GF-A_6P_TopMnt_Horizontal -> Customer_Connector:USB_C_Receptacle_6P_01
- L2: value 47uH 5040 -> 47uH 4030; footprint Inductor_SMD:L_Changjiang_FNR5040S -> Inductor_SMD:L_Changjiang_FNR4030S
- L6: footprint Inductor_SMD:L_Changjiang_FNR5040S -> Inductor_SMD:L_Changjiang_FNR4030S
- R1, R11, R13, R14, R2, R3, R6, R7, R8, R9: footprint Resistor_SMD:R_0402_1005Metric -> Resistor_SMD:R_0603_1608Metric
- R10, R4: footprint Resistor_SMD:R_1210_3225Metric -> Resistor_SMD:R_1206_3216Metric
- R12: renamed from R30; footprint (none) -> Resistor_SMD:R_0603_1608Metric
- R5: footprint Resistor_SMD:R_1206_3216Metric -> Resistor_SMD:R_0603_1608Metric
- renumbered C20 to C17, C7 to C18, C5 to C6, C13 to C7, D2 to D3, D3 to D4, L8 to L4, L4 to L8
Connections:
- net +12V: now also C11.1
- net GNDREF: now also C11.2, D2.1 (A1)
- net VCC: now also D2.2 (A2)
Other:
- moved on the sheet: D1, J1, R1, R2, R3

Commit message: Almost Finish
Parts:
- removed D2: PESD5V0 SOD-523, Diode_SMD:D_SOD-523, symbol Device:D_TVS
- added J2: Conn_01x10_Pin, Connector_PinHeader_2.54mm:PinHeader_1x10_P2.54mm_Horizontal, symbol Connector:Conn_01x10_Pin
- C11, C19, C20, C22, C8, C9: value 220uF 16V D8xL5 -> 100uF 16V D6.3xL5; footprint Capacitor_THT:CP_Radial_D8.0mm_P3.50mm -> Capacitor_THT:CP_Radial_D6.3mm_P2.50mm
Connections:
- net +12V: now also J2.10 (Pin_10), J2.8 (Pin_8), J2.9 (Pin_9)
- net -12V: now also J2.1 (Pin_1), J2.2 (Pin_2), J2.3 (Pin_3)
- net GNDREF: now also D1.1 (K), J2.4 (Pin_4), J2.5 (Pin_5), J2.6 (Pin_6), J2.7 (Pin_7); no longer R3.2
- net VCC: now also R3.1; no longer D1.2 (A)
- new net: D1.2 (A), R3.2
Other:
- moved on the sheet: D1, R3

Commit message: Update
Parts:
- removed C13, C2: 100uF 10V D5xL5, Capacitor_THT:CP_Radial_D4.0mm_P2.00mm, symbol Device:C_Polarized
- removed C17, C18, C20, C6, C7, C9: 100uF 16V D6.3xL5, Capacitor_THT:CP_Radial_D6.3mm_P2.50mm, symbol Device:C_Polarized
- added C13, C17, C2, C6, C7: 106 0805 25V X5R, Capacitor_SMD:C_0805_2012Metric, symbol Device:C
- added C9: 105 0603 25V X5R, Capacitor_SMD:C_0603_1608Metric, symbol Device:C
- C11, C19, C22, C8: value 100uF 16V D6.3xL5 -> 47uF 16V D5xL5; footprint Capacitor_THT:CP_Radial_D6.3mm_P2.50mm -> Capacitor_THT:CP_Radial_D5.0mm_P2.00mm
- C14: value 105 0603 25V X5R -> 106 0805 25V X5R; footprint Capacitor_SMD:C_0603_1608Metric -> Capacitor_SMD:C_0805_2012Metric
- J2: footprint Connector_PinHeader_2.54mm:PinHeader_1x10_P2.54mm_Horizontal -> Connector_PinHeader_2.54mm:PinHeader_1x10_P2.54mm_Vertical
- R10, R4: value 300mR 1206 -> 200mR 1206
- R11, R7: value 1k 0603 -> 499R 0603
- R12, R6: value 10.2k 0603 -> 5.1k 0603
- R13, R9: value 8.25k 0603 -> 5.1k 0603
- R14, R8: value 1k 0603 -> 604R 0603
Connections:
- net GNDREF: now also C14.2, C13.1, C17.2, C2.1, C6.1, C7.1, C9.2; no longer C14.1
- net U1_Vin: now also C2.2; no longer C3.2
- net U1_Vout: now also C6.2
- net U3_Vin: now also C13.2; no longer C14.2
- net U3_Vout: now also C14.1
- net at L3.2, L4.1: now also C3.2, C7.2
- net at L7.2, L8.1: now also C17.1, C9.1
Other:
- moved on the sheet: C1, C10, C11, C12, C19, C21, C22, C8, L1, L4, L5, L8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
